Commit message: ldlidar - add frame to the urdf, reference the node directly

File: mini_pupper_description/urdf/mini_pupper_description.urdf (robot description, URDF)
Before this commit: robot mini_pupper_description, 28 links, 27 joints
Links:
- added link lidar_frame, mass 0.001
Joints:
- added joint lidar_joint: type fixed, parent base_link, child lidar_frame, origin xyz=0.0 -0.05 0.03 rpy=0 0 1.57
